File: kicad/li_ion_charge.sch (KiCad schematic (older format))
At the start: 17 parts, among them P101 USB_B, P102 CONN_01X02, P103 CONN_01X02, U101 MCP73834-FCI/UN

Commit message: Final USB footprint and added a label to schematic
Parts:
- P101: footprint li_ion_charge_library:USB_Micro-B -> li_ion_charge_library:USB_Micro-B_10118193-0001LF
Changed lines of the file:
@@
 EESchema Schematic File Version 2
-LIBS:li_ion_charge-rescue
 LIBS:power
 LIBS:device
@@
 encoding utf-8
 Sheet 1 1
-Title ""
+Title "Single cell lithium ion battery charger using USB"
 Date ""
 Rev ""
-Comp ""
+Comp "Richard Memory"
 Comment1 ""
 Comment2 ""
@@
 F 0 "P101" V 2600 3550 50  0000 C CNN
 F 1 "USB_B" H 2850 3900 50  0000 C CNN
-F 2 "li_ion_charge_library:USB_Micro-B" V 2800 3450 50  0001 C CNN
+F 2 "li_ion_charge_library:USB_Micro-B_10118193-0001LF" V 2800 3450 50  0001 C CNN
 F 3 "http://portal.fciconnect.com/Comergent//fci/drawing/10118193.pdf" V 2800 3450 50  0001 C CNN
 F 4 "10118193-0001LF" V 2850 3550 60  0001 C CNN "MPN"
